File: Aft-PMAD-EthernetBridge/Aft-PMAD-EthernetBridge/Stepdown5VDC.kicad_sch (KiCad schematic)
At the start: 25 parts, among them M3 NVMFS6H836NLT1G, M4 NVMFS6H836NLT1G, U2 LM5148QRGYRQ1

Commit message: fix 5dc stepdown source from battery voltage to 24vdc source
Connections:
- net VBATT_50V4: no longer M3.5 (D), U2.12 (VIN)
- new net +24V: M3.5 (D), U2.12 (VIN)
