File: Aft-PMAD-EthernetBridge/Aft-PMAD-EthernetBridge/Stepdown24VDC.kicad_sch (KiCad schematic)
At the start: 25 parts, among them M1 NVMFS6H836NLT1G, M2 NVMFS6H836NLT1G, U1 LM5148QRGYRQ1

Commit message: update minor changes to 24vdc Step down (change resistor from 240K-ish to 10K) complete 3v3 stepdown
Parts:
- R7: value 287K -> 10K; MPN RC0402FR-07287KL -> RC0402FR-0710KL
Changed lines of the file:
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@@
 			)
 		)
-		(property "Value" "287K"
+		(property "Value" "10K"
 			(at 316.23 194.3099 0)
 			(show_name no)
@@
 			)
 		)
-		(property "MPN" "RC0402FR-07287KL"
+		(property "MPN" "RC0402FR-0710KL"
 			(at 316.23 201.9299 0)
 			(show_name no)
